File: expansion_board_EBAZ4205.kicad_pcb (KiCad board)
At the start: 2 copper layers, 86 x 55.8 mm, 56 parts, among them J1 INPUT, J2 CON_LIDAR, J3 CON_CAN, J4 DATA1, J5 DATA2, J6 DATA3_2.54, J7 DATA3, SW1 BTN1, SW2 BTN2, SW3 BTN3, SW4 BTN4, SW5 BTN5, U1 SN65HVD232, U2 NCP1117-3.3_SOT223

Commit message: update pdf
Parts:
- removed SW2: BTN2, Button_Switch_SMD:SW_SPST_CK_RS282G05A3
- removed SW3: BTN3, Button_Switch_SMD:SW_SPST_CK_RS282G05A3
- removed SW4: BTN4, Button_Switch_SMD:SW_SPST_CK_RS282G05A3
- removed SW5: BTN5, Button_Switch_SMD:SW_SPST_CK_RS282G05A3
- SW1: value BTN1 -> SW_DIP_x05; footprint Button_Switch_SMD:SW_SPST_CK_RS282G05A3 -> Button_Switch_SMD:SW_DIP_SPSTx05_Slide_6.7x14.26mm_W8.61mm_P2.54mm_LowProfile
- moved SW1 9.00 mm to (119.8, 57.9)
- moved R17 3.85 mm to (124.9, 50.0), turned to -90 degrees
- moved R13 3.70 mm to (114.7, 49.9), turned to -90 degrees
- moved J4 2.00 mm to (106.0, 31.5)
- moved R16 1.85 mm to (122.4, 50.0), turned to -90 degrees
- moved R14 1.60 mm to (117.1, 49.9), turned to -90 degrees
- moved J5 1.00 mm to (129.0, 31.5)
- turned R15 to -90 degrees
- renumbered JP2 to 120, D2 to 12V, D1 to 3V3, D3 to 5V, JP1 to 5V, TP4 to CANH, TP5 to CANL, TP1 to PWM, TP2 to RX, TP3 to TX
Connections:
- SW1 pad 2: /L16 -> +3V3
Routing:
- net +3V3: track 142.2 -> 138.0 mm
- net /H20: track 24.5 -> 27.9 mm
- net /M18: track 28.5 -> 31.8 mm
- net /M20: track 23.9 -> 26.5 mm
- net /J18: track 24.2 -> 26.7 mm
- net /L16: track 23.4 -> 25.2 mm
- net /C20: track 50.7 -> 51.7 mm
- net /B19: track 52.0 -> 52.9 mm
- net /F20: track 10.1 -> 11.0 mm
- net /A20: track 52.7 -> 53.6 mm
- net GND: vias 25 -> 47
Other:
- board text added: "3V3"
- board text added: "5V"
- board text added: "EBAZ4205 Expansion board REV 1.0 https://github.com/kingovchouffe"
- board text added: "G19"
- board text added: "G20"
- board text added: "H20"
- board text added: "J18"
- board text added: "J19"
- board text added: "K18"
- board text added: "K19"
- board text added: "L17"
- board text added: "L18"
- board text added: "L19"
- board text added: "L20"
- board text added: "LED"
- board text added: "M18"
- board text added: "M20"
- board text added: "N17"
- board text added: "P19"
- board text added: "P20"
- board text added: "R18"
- board text added: "R19"
- board text added: "RGB"
- board text added: "T19"
- board text added: "T20"
- board text added: "U19"
- board text added: "U20"
- board text added: "V20"
