File: expansion_board_EBAZ4205.kicad_sch (KiCad schematic)
At the start: 56 parts, among them J1 INPUT, J2 CON_LIDAR, J3 CON_CAN, J4 DATA1, J5 DATA2, J6 DATA3_2.54, J7 DATA3, SW1 BTN1, SW2 BTN2, SW3 BTN3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

Commit message: update pdf
Parts:
- removed SW1: BTN1, Button_Switch_SMD:SW_SPST_CK_RS282G05A3, symbol Switch:SW_Push
- removed SW2: BTN2, Button_Switch_SMD:SW_SPST_CK_RS282G05A3, symbol Switch:SW_Push
- removed SW3: BTN3, Button_Switch_SMD:SW_SPST_CK_RS282G05A3, symbol Switch:SW_Push
- removed SW4: BTN4, Button_Switch_SMD:SW_SPST_CK_RS282G05A3, symbol Switch:SW_Push
- removed SW5: BTN5, Button_Switch_SMD:SW_SPST_CK_RS282G05A3, symbol Switch:SW_Push
- added SW1: SW_DIP_x05, Button_Switch_SMD:SW_DIP_SPSTx05_Slide_6.7x14.26mm_W8.61mm_P2.54mm_LowProfile, symbol Switch:SW_DIP_x05
Connections:
- net +3V3: now also SW1.1, SW1.2, SW1.3, SW1.4, SW1.5
- net H20: now also SW1.6
- net J18: now also SW1.7
- net L16: now also SW1.10
- net M18: now also SW1.9
- net M20: now also SW1.8
Other:
- moved on the sheet: D10, D6, D7, D8, D9, H1, H3, H4, J4, J5, J6, J7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
